File: RC5-preamp-board.sch (KiCad schematic (older format))
At the start: 17 parts, among them P1 RAW_DC, P10 CTL_OUT, P2 VCC, P3 VCC, P4 VCC, P5 VCC, P6 VCC, P8 INPUTS, P9 UI_OUT, U1 NCP1117DT50RKG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

Commit message: Added additional current limitation comments to schematic and increased max. sink per Arduino spec.
Other:
- note added: "20mA per pin max."
- note added: "Collective maximum current output is 150 mA."
- note removed: "10mA per pin max."
Changed lines of the file:
@@
 Sheet 1 2
 Title "RC5 remote control board"
-Date "20 apr 2015"
+Date "24 apr 2015"
 Rev "1.0"
 Comp "Mithat Konar"
@@
 63 98 05 E1 6B C4 72 91 8E EA 95 27 8C 4B 0B 6B 30 6B 95 2D 08 DF 47 79 14 D8 40 20 A9 90 96 2D
 E1 E7 3D C6 74 F3 E0 6E B9 00 E4 0E CC EC 2A 00 9E 03 F9 2E 43 53 93 3B E7 B1 3D FE 0F E4 2C B5
-B8 3A B8 3B 5D 00 00 00 00 49 45 4E 44 AE 42 60 82 A1 $EndBitmap
+B8 3A B8 3B 5D 00 00 00 00 49 45 4E 44 AE 42 60 82 00 $EndBitmap
 EndData
 $EndBitmap
@@
 	3700 1050 4500 1050
 Text Notes 8450 3800 2    60   ~ 0
-10mA per pin max.
+20mA per pin max.
 Wire Wire Line
 	9150 1100 9150 2300
+Text Notes 8400 4450 2    60   ~ 0
+20mA per pin max.
+Text Notes 7750 4900 0    60   ~ 0
+Collective maximum current output is 150 mA.
 $EndSCHEMATC
