File: arduino-pcb.sch (KiCad schematic (older format))
At the start: 12 parts, among them P201 FTDI basic, SW201 Reset, U201 ATMEGA328P-PU, X201 CSTLS16M0X53-B0

Commit message: PCB placed, routability confirmed.
Parts:
- removed R203, R204: opt, mfk-R_0.25W_RN55_vert, symbol R
- P201: value FTDI basic -> FTDI Basic; footprint (none) -> mfk-SIL-6
- R201, R202: footprint mfk-R_0.25W_RN55_vert -> mfk-R_0.25W_RN55
- SW201: footprint mfk-SW_PUSH_6MM -> mfk-SW_PUSH_6x3.5mm
- U201: footprint DIL28 -> mfk-DIP-28_300_rnd
Other:
- note removed: "Optional pullups for I2C"
Changed lines of the file:
@@
 LIBS:mfk_atmel
 LIBS:mfk_opto
+LIBS:mfk_vreg
 LIBS:power
 LIBS:device
@@
 Sheet 2 2
 Title "Arduino ATMEGA328-PU subcircuit"
-Date "17 apr 2015"
+Date "18 apr 2015"
 Rev ""
 Comp "Mithat Konar"
@@
 F 0 "R201" V 3580 3000 40  0000 C CNN
 F 1 "10K" V 3507 3001 40  0000 C CNN
-F 2 "mfk-R_0.25W_RN55_vert" V 3430 3000 30  0001 C CNN
+F 2 "mfk-R_0.25W_RN55" V 3430 3000 30  0001 C CNN
 F 3 "~" H 3500 3000 30  0000 C CNN
 	1    3500 3000
@@
 F 0 "SW201" H 3500 3900 50  0000 C CNN
 F 1 "Reset" H 3500 3670 50  0000 C CNN
-F 2 "mfk-SW_PUSH_6MM" H 3500 3750 60  0001 C CNN
+F 2 "mfk-SW_PUSH_6x3.5mm" H 3500 3750 60  0001 C CNN
 F 3 "~" H 3500 3750 60  0000 C CNN
 	1    3500 3750
@@
 F 0 "R202" V 7180 2350 40  0000 C CNN
 F 1 "330" V 7107 2351 40  0000 C CNN
-F 2 "mfk-R_0.25W_RN55_vert" V 7030 2350 30  0001 C CNN
+F 2 "mfk-R_0.25W_RN55" V 7030 2350 30  0001 C CNN
 F 3 "~" H 7100 2350 30  0000 C CNN
 	1    7100 2350
@@
 	0    1    1    0
 $EndComp
-$Comp
-L R R204
-U 1 1 553171BF
-P 8250 2350
-F 0 "R204" V 8330 2350 40  0000 C CNN
-F 1 "opt" V 8257 2351 40  0000 C CNN
-F 2 "mfk-R_0.25W_RN55_vert" V 8180 2350 30  0001 C CNN
-F 3 "~" H 8250 2350 30  0000 C CNN
-	1    8250 2350
-	1    0    0    -1
-$EndComp
-$Comp
-L R R203
-U 1 1 553171C5
-P 8050 2350
-F 0 "R203" V 8130 2350 40  0000 C CNN
-F 1 "opt" V 8057 2351 40  0000 C CNN
-F 2 "mfk-R_0.25W_RN55_vert" V 7980 2350 30  0001 C CNN
-F 3 "~" H 8050 2350 30  0000 C CNN
-	1    8050 2350
-	1    0    0    -1
-$EndComp
-Text Notes 8450 2700 1    40   ~ 0
-Optional pullups for I2C
 Wire Wire Line
 	4300 4200 4600 4200
@@
 	7450 4800 8600 4800
 Wire Wire Line
-	8250 1700 8250 2100
-Wire Wire Line
-	8050 2100 8050 2050
-Wire Wire Line
 	6800 3550 7500 3550
 Wire Wire Line
@@
 Wire Wire Line
 	6800 3850 7550 3850
-Wire Wire Line
-	8050 2900 8050 2600
 Wire Wire Line
 	7450 4150 7450 4050
@@
 Text HLabel 8600 6000 2    60   BiDi ~ 0
 RXI
-Text Label 8050 2900 1    60   ~ 0
-A5
-Wire Wire Line
-	8250 2900 8250 2600
-Text Label 8250 2900 1    60   ~ 0
-A4
-Wire Wire Line
-	8050 2050 8250 2050
-Connection ~ 8250 2050
-Text Label 8250 1700 3    60   ~ 0
-V_VCC
 Text Label 3500 2450 3    60   ~ 0
 V_VCC
@@
 F 0 "U201" H 5050 5700 40  0000 L BNN
 F 1 "ATMEGA328P-PU" H 6650 3050 40  0000 R BNN
-F 2 "DIL28" H 5800 4450 30  0000 C CIN
+F 2 "mfk-DIP-28_300_rnd" H 5800 4450 30  0001 C CIN
 F 3 "~" H 5800 4450 60  0000 C CNN
 	1    5850 4450
@@
 P 5750 1400
 F 0 "P201" V 5700 1400 60  0000 C CNN
-F 1 "FTDI basic" V 5800 1400 60  0000 C CNN
-F 2 "" H 5750 1400 60  0000 C CNN
+F 1 "FTDI Basic" V 5800 1400 60  0000 C CNN
+F 2 "mfk-SIL-6" H 5750 1400 60  0001 C CNN
 F 3 "" H 5750 1400 60  0000 C CNN
 	1    5750 1400
@@
 D8
 $Comp
-L DGND #PWR014
+L DGND #PWR013
 U 1 1 553228EE
 P 5500 1900
-F 0 "#PWR014" H 5500 1900 40  0001 C CNN
+F 0 "#PWR013" H 5500 1900 40  0001 C CNN
 F 1 "DGND" H 5500 1830 40  0000 C CNN
 F 2 "" H 5500 1900 60  0000 C CNN
@@
 $EndComp
 $Comp
-L DGND #PWR015
+L DGND #PWR014
 U 1 1 55322907
 P 7100 3100
-F 0 "#PWR015" H 7100 3100 40  0001 C CNN
+F 0 "#PWR014" H 7100 3100 40  0001 C CNN
 F 1 "DGND" H 7100 3030 40  0000 C CNN
 F 2 "" H 7100 3100 60  0000 C CNN
@@
 $EndComp
 $Comp
-L DGND #PWR016
+L DGND #PWR015
 U 1 1 55322916
 P 4500 4850
-F 0 "#PWR016" H 4500 4850 40  0001 C CNN
+F 0 "#PWR015" H 4500 4850 40  0001 C CNN
 F 1 "DGND" H 4500 4780 40  0000 C CNN
 F 2 "" H 4500 4850 60  0000 C CNN
@@
 $EndComp
 $Comp
-L DGND #PWR017
+L DGND #PWR016
 U 1 1 55322925
 P 4850 4650
-F 0 "#PWR017" H 4850 4650 40  0001 C CNN
+F 0 "#PWR016" H 4850 4650 40  0001 C CNN
 F 1 "DGND" H 4850 4580 40  0000 C CNN
 F 2 "" H 4850 4650 60  0000 C CNN
@@
 $EndComp
 $Comp
-L DGND #PWR018
+L DGND #PWR017
 U 1 1 55322934
 P 4850 5250
-F 0 "#PWR018" H 4850 5250 40  0001 C CNN
+F 0 "#PWR017" H 4850 5250 40  0001 C CNN
 F 1 "DGND" H 4850 5180 40  0000 C CNN
 F 2 "" H 4850 5250 60  0000 C CNN
@@
 $EndComp
 $Comp
-L DGND #PWR019
+L DGND #PWR018
 U 1 1 55322943
 P 4500 5550
-F 0 "#PWR019" H 4500 5550 40  0001 C CNN
+F 0 "#PWR018" H 4500 5550 40  0001 C CNN
 F 1 "DGND" H 4500 5480 40  0000 C CNN
 F 2 "" H 4500 5550 60  0000 C CNN
@@
 $EndComp
 $Comp
-L DGND #PWR020
+L DGND #PWR019
 U 1 1 55322952
 P 3500 4100
-F 0 "#PWR020" H 3500 4100 40  0001 C CNN
+F 0 "#PWR019" H 3500 4100 40  0001 C CNN
 F 1 "DGND" H 3500 4030 40  0000 C CNN
 F 2 "" H 3500 4100 60  0000 C CNN
@@
 $EndComp
 $Comp
-L DGND #PWR021
+L DGND #PWR020
 U 1 1 55326F97
 P 4100 4000
-F 0 "#PWR021" H 4100 4000 40  0001 C CNN
+F 0 "#PWR020" H 4100 4000 40  0001 C CNN
 F 1 "DGND" H 4100 3930 40  0000 C CNN
 F 2 "" H 4100 4000 60  0000 C CNN
